File: hardware/fk-naturalist.sch (KiCad schematic (older format))
At the start: 89 parts, among them J1 MICRO-USB, J2 CONN_01X03, J3 Conn_01x10, J4 Conn_01x02, J5 Conn_01x01, J6 CONN-HDR-2x5, J8 Conn_01x01, M1 MOUNT_HOLE, M2 MOUNT_HOLE, M3 MOUNT_HOLE, M4 MOUNT_HOLE, Q1 2N7002LT1G, Q2 2N7002LT1G, Q3 2N7002LT1G, Q4 2N7002LT1G, SW1 SPNO, U1 ATSAMD21G18A-AU, U101 TSL2591, U102 MPL3115A2, U103 BNO055, U104 SHT31, U2 MCP1700T-XXX2E, U3 MAX4466, U4 S25FL1xxK0XM, Y1 FC-135, Y101 FC-135

Commit message: Making the schematic more organized for a presentation.
Connections:
- wire segments 295 -> 349
Other:
- note added: "ATSAMD21D\n"
- note added: "BNO055 IMU"
- note added: "HEADERS"
- note added: "LEDS"
- note added: "MAX4466 MICROPHONE"
- note added: "MPL3115A2"
- note added: "PULLUPS"
- note added: "SERIAL FLASH"
- note added: "SHT31"
- note added: "TSL2591"
- note added: "USB"
- moved on the sheet: C1, C10, C101, C102, C103, C104, C105, C106, C107, C108, C109, C11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
