File: hardware/main-board/fk-naturalist.sch (KiCad schematic (older format))
At the start: 136 parts, among them J1 Conn_01x11, J10 S2B-PH-SM4-TB, J11 RF-SMA-EDGE, J2 Conn_01x05, J3 Conn_01x04, J4 Conn_01x02, J5 Conn_01x03, J6 Conn_01x05, J7 CONN-HDR-2x5, J8 Conn_01x09, J9 MICRO-USB, M1 MOUNT_HOLE, M3 MOUNT_HOLE, M4 MOUNT_HOLE, M6 MOUNT_HOLE, M7 MICROSD, Q1 2N7002LT1G, Q2 2N7002LT1G, Q3 2N7002LT1G, Q4 2N7002LT1G, Q5 2N7002LT1G, SW1 SPNO, SW2 SPNO, U1 ATWINC1500-MR210PA, U10 FGPMMOPA6H, U101 TSL2591, U102 MPL3115A2, U103 BNO055, U104 SHT31, U11 MAX1704XX, U2 ATSAMD21G18A-AU, U3 SPH0645, U4 24AA02E64, U5 S25FL116K0XMFI041, U6 BQ24074RGTT, U7 PCF8523, U8 MCP1700T-3302E/MB, U9 ISL8541x, Y1 FC-135, Y101 FC-135, Y2 FC-135

Commit message: Remove sensors from main board. Add connector.
Parts:
- removed C101, C13: 1uF, RocketScreamKicadLibrary:CAP-0603, symbol CAPACITOR-CERAMIC
- removed C102, C103, C109: 100nF, RocketScreamKicadLibrary:CAP-0603, symbol CAPACITOR-CERAMIC
- removed C104: 10uF, RocketScreamKicadLibrary:CAP-0603, symbol CAPACITOR-CERAMIC
- removed C15: 220pF, RocketScreamKicadLibrary:CAP-0603, symbol CAPACITOR-CERAMIC
- removed J1: Conn_01x11, Socket_Strips:Socket_Strip_Straight_1x11_Pitch2.54mm, symbol Conn_01x11
- removed J2: Conn_01x05, Socket_Strips:Socket_Strip_Straight_1x05_Pitch2.54mm, symbol Conn_01x05
- removed J3: Conn_01x04, Socket_Strips:Socket_Strip_Straight_1x04_Pitch2.54mm, symbol Conn_01x04
- removed R11: 10K, RocketScreamKicadLibrary:RES-0603, symbol RESISTOR
- removed R12: 68R, RocketScreamKicadLibrary:RES-0603, symbol RESISTOR
- removed U101: TSL2591, conservify:TSL2591, symbol TSL2591
- removed U102: MPL3115A2, conservify:DFN-8-1EP_5x2.55mm_Pitch1.25mm_98ASA002260D, symbol MPL3115A2
- removed U104: SHT31, conservify:SHT3x, symbol SHT31
- removed U3: SPH0645, conservify:SPH0645LM4H-B, symbol SPH0645
- added J1: Conn_01x07, conservify:Molex_CLIK-Mate_502386-0770_1x07_P1.25mm_Horizontal, symbol Conn_01x07
Connections:
- wire segments 501 -> 441
- no-connect marks 37 -> 33
Other:
- note removed: "AUDIO"
- note removed: "MPL3115A2"
- note removed: "SHT31"
- note removed: "TSL2591"
- moved on the sheet: C105, C106, C107, C108, C11, R101, R102, R103, U103, U4, Y101

Commit message: Adding fiducials.
Parts:
- added M2, M5, M8: FIDUCIAL, Fiducials:Fiducial_0.75mm_Dia_1.5mm_Outer, symbol FIDUCIAL
- BT1: Critical (none) -> (none); MFN (none) -> Harwin; MFP (none) -> S8411-45R; Notes (none) -> (none); Package (none) -> (none); Source (none) -> ANY; Subsystem (none) -> (none)
- C1, C12, C21, C23, C27, C29, C6: Critical (none) -> (none); MFN (none) -> Taiyo Yuden; MFP (none) -> UMK107BJ105KA-T; Notes (none) -> (none); Package (none) -> (none); Source (none) -> ANY; Subsystem (none) -> (none)
- C10, C19, C20, C25: Critical (none) -> (none); MFN (none) -> AVX; MFP (none) -> 0603ZD475MAT2A; Notes (none) -> (none); Package (none) -> (none); Source (none) -> ANY; Subsystem (none) -> (none)
- C105, C107: Critical (none) -> (none); MFN (none) -> AVX; MFP (none) -> 06035A220JAT2A; Notes (none) -> (none); Package (none) -> (none); Source (none) -> ANY; Subsystem (none) -> (none)
- C106, C108, C11, C18, C26, C5, C7, C8, C9: Critical (none) -> (none); MFN (none) -> Murata Electronics; MFP (none) -> GRM188R71H104KA93D; Notes (none) -> (none); Package (none) -> (none); Source (none) -> ANY; Subsystem (none) -> (none)
- C14: Critical (none) -> (none); MFN (none) -> KEMET; MFP (none) -> C0603C472K9RACTU; Notes (none) -> (none); Package (none) -> (none); Source (none) -> ANY; Subsystem (none) -> (none)
- C22, C24, C31, C32: Critical (none) -> (none); MFN (none) -> Taiyo Yuden; MFP (none) -> LMK107BBJ106KALT; Notes (none) -> (none); Package (none) -> (none); Source (none) -> ANY; Subsystem (none) -> (none)
- C28: Critical (none) -> (none); MFN (none) -> AVX; MFP (none) -> 0603YC103K4T2A; Notes (none) -> (none); Package (none) -> (none); Source (none) -> ANY; Subsystem (none) -> (none)
- C3, C4: Critical (none) -> (none); MFN (none) -> AVX; MFP (none) -> 06035A180JAT2A; Notes (none) -> (none); Package (none) -> (none); Source (none) -> ANY; Subsystem (none) -> (none)
- C30: Critical (none) -> (none); MFN (none) -> AVX; MFP (none) -> 06035C101KAT2A; Notes (none) -> (none); Package (none) -> (none); Source (none) -> ANY; Subsystem (none) -> (none)
- D1, D4: Critical (none) -> (none); MFN (none) -> Lite-On; MFP (none) -> LTST-C190KFKT; Notes (none) -> (none); Package (none) -> (none); Source (none) -> ANY; Subsystem (none) -> (none)
- D10, D11: Critical (none) -> (none); MFN (none) -> Lite-On; MFP (none) -> LTST-C190KRKT; Notes (none) -> (none); Package (none) -> (none); Source (none) -> ANY; Subsystem (none) -> (none)
- D2, D9: Critical (none) -> (none); MFN (none) -> Lite-On; MFP (none) -> LTST-C190KGKT; Notes (none) -> (none); Package (none) -> (none); Source (none) -> ANY; Subsystem (none) -> (none)
- D3, D5: Critical (none) -> (none); MFN (none) -> Lite-On; MFP (none) -> LTST-C190KSKT; Notes (none) -> (none); Package (none) -> (none); Source (none) -> ANY; Subsystem (none) -> (none)
- D6: Critical (none) -> (none); MFN (none) -> Lite-On; MFP (none) -> LTST-C191TBKT; Notes (none) -> (none); Package (none) -> (none); Source (none) -> ANY; Subsystem (none) -> (none)
- D7: Critical (none) -> (none); MFN (none) -> Nexperia; MFP (none) -> PMEG3020CPA,115; Notes (none) -> (none); Package (none) -> (none); Source (none) -> ANY; Subsystem (none) -> (none)
- D8: symbol PRTR5V0U2X -> PRTR5V0U2X-RESCUE-fk-naturalist; Critical (none) -> (none); MFN (none) -> Nexperia; MFP (none) -> PRTR5V0U2X,215; Notes (none) -> (none); Package (none) -> (none); Source (none) -> ANY; Subsystem (none) -> (none)
- F1: Critical (none) -> (none); MFN (none) -> Bourns; MFP (none) -> MF-PSMF050X-2; Notes (none) -> (none); Package (none) -> (none); Source (none) -> ANY; Subsystem (none) -> (none)
- J1: Critical (none) -> (none); MFN (none) -> Molex; MFP (none) -> 502386-0770; Notes (none) -> (none); Package (none) -> (none); SPN1 (none) -> 538-502386-0770; Source (none) -> ANY; Subsystem (none) -> (none); Supplier1 (none) -> mouser
- J10: Critical (none) -> (none); MFN (none) -> JST; MFP (none) -> S2B-PH-SM4-TB(LF)(SN); Notes (none) -> (none); Package (none) -> (none); Source (none) -> ANY; Subsystem (none) -> (none)
- J11: Critical (none) -> (none); MFN (none) -> (none); MFP (none) -> (none); Notes (none) -> (none); Package (none) -> (none); Source (none) -> ANY; Subsystem (none) -> (none)
- J4, J8, M1, M3, M4, M6: Critical (none) -> (none); MFN (none) -> (none); MFP (none) -> (none); Notes (none) -> (none); Package (none) -> (none); SPN1 (none) -> (none); Source (none) -> ANY; Subsystem (none) -> (none); Supplier1 (none) -> (none)
- J5: Critical (none) -> (none); MFN (none) -> Molex; MFP (none) -> 502382-0370; Notes (none) -> (none); Package (none) -> (none); Source (none) -> ANY; Subsystem (none) -> (none)
- J6: Critical (none) -> (none); MFN (none) -> Molex; MFP (none) -> 502382-0570; Notes (none) -> (none); Package (none) -> (none); Source (none) -> ANY; Subsystem (none) -> (none)
- J7: Critical (none) -> (none); MFN (none) -> Amphenol FCI; MFP (none) -> 20021121-00010C4LF; Notes (none) -> (none); Package (none) -> (none); Source (none) -> ANY; Subsystem (none) -> (none)
- J9: Critical (none) -> (none); MFN (none) -> Hirose Connector; MFP (none) -> ZX62D-B-5PA8(30); Notes (none) -> (none); Package (none) -> (none); Source (none) -> ANY; Subsystem (none) -> (none)
- L1, L2: symbol INDUCTOR -> INDUCTOR-RESCUE-fk-naturalist; Critical (none) -> (none); MFN (none) -> Murata Electronics; MFP (none) -> BLM18KG221SN1D; Notes (none) -> (none); Package (none) -> (none); Source (none) -> ANY; Subsystem (none) -> (none)
- L5: symbol INDUCTOR -> INDUCTOR-RESCUE-fk-naturalist; Critical (none) -> (none); MFN (none) -> Wurth Electronics; MFP (none) -> 74404064220; Notes (none) -> (none); Package (none) -> (none); Source (none) -> ANY; Subsystem (none) -> (none)
- M7: Critical (none) -> (none); MFN (none) -> 3M; MFP (none) -> 2908-05WB-MG; Notes (none) -> (none); Package (none) -> (none); Source (none) -> ANY; Subsystem (none) -> (none)
- Q1, Q2, Q3, Q4, Q5: Critical (none) -> (none); MFN (none) -> ON Semiconductor; MFP (none) -> 2N7002LT1G; Notes (none) -> (none); Package (none) -> (none); Source (none) -> ANY; Subsystem (none) -> (none)
- R1, R2, R23, R38, R44: Critical (none) -> (none); MFN (none) -> Yageo; MFP (none) -> RC0603FR-07100KL; Notes (none) -> (none); Package (none) -> (none); Source (none) -> ANY; Subsystem (none) -> (none)
- R10, R30, R9: Critical (none) -> (none); MFN (none) -> Yageo; MFP (none) -> RC0603FR-07330RL; Notes (none) -> (none); Package (none) -> (none); Source (none) -> ANY; Subsystem (none) -> (none)
- R101, R102, R103, R17, R32, R34, R6, R8: Critical (none) -> (none); MFN (none) -> Yageo; MFP (none) -> RC0603FR-0710KL; Notes (none) -> (none); Package (none) -> (none); Source (none) -> ANY; Subsystem (none) -> (none)
- R18, R19, R20, R25, R3, R33: Critical (none) -> (none); MFN (none) -> Yageo; MFP (none) -> RC0603FR-072K2L; Notes (none) -> (none); Package (none) -> (none); Source (none) -> ANY; Subsystem (none) -> (none)
- R21: Critical (none) -> (none); MFN (none) -> Panasonic; MFP (none) -> ERJ-PA3F1181V; Notes (none) -> (none); Package (none) -> (none); Source (none) -> ANY; Subsystem (none) -> (none)
- R22: Critical (none) -> (none); MFN (none) -> Panasonic Industrial Devices; MFP (none) -> ERJ-3EKF4642V; Notes (none) -> (none); Package (none) -> (none); Source (none) -> ANY; Subsystem (none) -> (none)
- R24: Critical (none) -> (none); MFN (none) -> Panasonic; MFP (none) -> ERJ-S03F2941V; Notes (none) -> (none); Package (none) -> (none); Source (none) -> ANY; Subsystem (none) -> (none)
- R26, R27, R35, R36, R42, R43: Critical (none) -> (none); MFN (none) -> Yageo; MFP (none) -> AF0603JR-074K7L; Notes (none) -> (none); Package (none) -> (none); Source (none) -> ANY; Subsystem (none) -> (none)
- R31: Critical (none) -> (none); MFN (none) -> Yageo; MFP (none) -> RC0603FR-071ML; Notes (none) -> (none); Package (none) -> (none); Source (none) -> ANY; Subsystem (none) -> (none)
- R37, R39, R4, R40, R5: Critical (none) -> (none); MFN (none) -> Yageo; MFP (none) -> RC0603FR-071KL; Notes (none) -> (none); Package (none) -> (none); Source (none) -> ANY; Subsystem (none) -> (none)
- R41: Critical (none) -> (none); MFN (none) -> Yageo; MFP (none) -> RC0603FR-07180RL; Notes (none) -> (none); Package (none) -> (none); Source (none) -> ANY; Subsystem (none) -> (none)
- R45: Critical (none) -> (none); MFN (none) -> Yageo; MFP (none) -> RC0603FR-0722KL; Notes (none) -> (none); Package (none) -> (none); Source (none) -> ANY; Subsystem (none) -> (none)
- SW1, SW2: Critical (none) -> (none); MFN (none) -> Wurth Electronics; MFP (none) -> 434331045822; Notes (none) -> (none); Package (none) -> (none); Source (none) -> ANY; Subsystem (none) -> (none)
- U1: Critical (none) -> (none); MFN (none) -> Microchip Technology; MFP (none) -> ATWINC1500-MR210UB; Notes (none) -> (none); Package (none) -> (none); Source (none) -> ANY; Subsystem (none) -> (none)
- U10: Critical (none) -> (none); MFN (none) -> GlobalTop Technology; MFP (none) -> FGPMMOPA6H; Notes (none) -> (none); Package (none) -> (none); SPN1 (none) -> (none); Source (none) -> ANY; Subsystem (none) -> (none)
- U103: Critical (none) -> (none); MFN (none) -> Bosch Sensortec; MFP (none) -> BNO055; Notes (none) -> (none); Package (none) -> (none); Source (none) -> ANY; Subsystem (none) -> (none)
- U11: Critical (none) -> (none); MFN (none) -> Maxim Integrated; MFP (none) -> MAX17043G+U; Notes (none) -> (none); Package (none) -> (none); Source (none) -> ANY; Subsystem (none) -> (none)
- U2: Critical (none) -> (none); MFN (none) -> Microchip Technology / Atmel; MFP (none) -> ATSAMD21G18A-AU; Notes (none) -> (none); Package (none) -> (none); Source (none) -> ANY; Subsystem (none) -> (none)
- U4: Critical (none) -> (none); MFN (none) -> Microchip Technology; MFP (none) -> 24AA02E64T-I/OT; Notes (none) -> (none); Package (none) -> (none); Source (none) -> ANY; Subsystem (none) -> (none)
- U5: Critical (none) -> (none); MFN (none) -> Cypress Semiconductor; MFP (none) -> S25FL116K0XMFI041; Notes (none) -> (none); Package (none) -> (none); Source (none) -> ANY; Subsystem (none) -> (none)
- U6: Critical (none) -> (none); MFN (none) -> Texas Instruments; MFP (none) -> BQ24074RGTT; Notes (none) -> (none); Package (none) -> (none); Source (none) -> ANY; Subsystem (none) -> (none)
- U7: Critical (none) -> (none); MFN (none) -> NXP Semiconductors; MFP (none) -> PCF8523T/1,118; Notes (none) -> (none); Package (none) -> (none); Source (none) -> ANY; Subsystem (none) -> (none)
- U8: Critical (none) -> (none); MFN (none) -> Microchip Technology; MFP (none) -> MCP1700T-3302E/MB; Notes (none) -> (none); Package (none) -> (none); Source (none) -> ANY; Subsystem (none) -> (none)
- U9: Critical (none) -> (none); MFN (none) -> Renesas / Intersil; MFP (none) -> ISL85415FRZ; Notes (none) -> (none); Package (none) -> (none); Source (none) -> ANY; Subsystem (none) -> (none)
- Y1, Y101, Y2: Critical (none) -> (none); MFN (none) -> Epson Timing; MFP (none) -> FC-135 32.7680KA-A3; Notes (none) -> (none); Package (none) -> (none); Source (none) -> ANY; Subsystem (none) -> (none)

Commit message: Adding fiducials to the bottom.
Parts:
- added M10, M11, M9: FIDUCIAL, Fiducials:Fiducial_0.75mm_Dia_1.5mm_Outer, symbol FIDUCIAL
