File: hardware/main-board/fk-naturalist.sch (KiCad schematic (older format))
At the start: 119 parts, among them J1 Conn_01x07, J10 S2B-PH-SM4-TB, J11 RF-SMA-EDGE, J4 Conn_01x02, J5 Conn_01x03, J6 Conn_01x05, J7 CONN-HDR-2x5, J8 Conn_01x09, J9 MICRO-USB, M1 MOUNT_HOLE, M10 FIDUCIAL, M11 FIDUCIAL, M2 FIDUCIAL, M3 MOUNT_HOLE, M4 MOUNT_HOLE, M5 FIDUCIAL, M6 MOUNT_HOLE, M7 MICROSD, M8 FIDUCIAL, M9 FIDUCIAL, Q1 2N7002LT1G, Q5 2N7002LT1G, SW1 SPNO, SW2 SPNO, U1 ATWINC1500-MR210PA, U10 FGPMMOPA6H, U103 BNO055, U11 MAX1704XX, U2 ATSAMD21G18A-AU, U3 SK6812, U4 24AA02E64, U5 S25FL116K0XMFI041, U6 BQ24074RGTT, U7 PCF8523, U8 MCP1700T-3302E/MB, U9 ISL8541x, Y1 FC-135, Y101 FC-135, Y2 FC-135

Commit message: Consistent part values across our schematics.
Parts:
- R1, R2, R38, R44: value 100k -> 100K
- R37, R39, R4, R40, R5: value 1k -> 1K

Commit message: Part updates.
Parts:
- BT1: value Battery_Cell -> BATTERY_CELL
- J7: value CONN-HDR-2x5 -> CONN_02x05_SWD
Changed lines of the file:
@@
 P 6100 9900
 F 0 "J7" H 6100 10250 60 0000 C CNN
-F 1 "CONN-HDR-2x5" H 6100 9500 60 0001 C CNN
+F 1 "CONN_02x05_SWD" H 6100 9500 60 0001 C CNN
 F 2 "conservify:HDR_2x5_Pitch1.27mm_SMD_JTAG_SWD" H 6100 9400 60 0001 C CNN
 F 3 "" H 6100 9750 60 0000 C CNN
@@
 P 12200 6550
 F 0 "BT1" H 12300 6650 50 0000 L CNN
-F 1 "Battery_Cell" H 12300 6550 50 0000 L CNN
+F 1 "BATTERY_CELL" H 12300 6550 50 0000 L CNN
 F 2 "conservify:BAT_CR1210" V 12200 6610 50 0001 C CNN
 F 3 "" V 12200 6610 50 0001 C CNN

Commit message: Fix SK6812.
Parts:
- J7: footprint conservify:HDR_2x5_Pitch1.27mm_SMD_JTAG_SWD -> conservify:HDR_02x05_Pitch1.27mm_SMD_SWD

Commit message: Main board is now same as fk-core.
Parts:
- removed C105, C107: 22pF, conservify:CAP-0603, symbol RocketScreamKicadLibrary:CAPACITOR-CERAMIC
- removed C106, C108, C26: 100nF, conservify:CAP-0603, symbol RocketScreamKicadLibrary:CAPACITOR-CERAMIC
- removed C21, C23, C29: 1uF, conservify:CAP-0603, symbol RocketScreamKicadLibrary:CAPACITOR-CERAMIC
- removed C25: 4.7uF, conservify:CAP-0603, symbol RocketScreamKicadLibrary:CAPACITOR-CERAMIC
- removed C30: 100pF, conservify:CAP-0603, symbol RocketScreamKicadLibrary:CAPACITOR-CERAMIC
- removed C31, C32: 10uF, conservify:CAP-0603, symbol RocketScreamKicadLibrary:CAPACITOR-CERAMIC
- removed J1: Conn_01x07, conservify:Molex_CLIK-Mate_502386-0770_1x07_P1.25mm_Horizontal, symbol fk-naturalist-rescue:Conn_01x07
- removed J4: Conn_01x02, conservify:SJ_OPEN, symbol fk-naturalist-rescue:Conn_01x02
- removed J5: Conn_01x03, conservify:Molex_CLIK-Mate_502382-0370_1x03_P1.25mm_Vertical, symbol fk-naturalist-rescue:Conn_01x03
- removed J8: Conn_01x09, conservify:Socket_Strip_Straight_1x09_Pitch2.54mm, symbol fk-naturalist-rescue:Conn_01x09
- removed L5: 22uH, conservify:WURTH_L_6.0x6.0, symbol fk-naturalist-rescue:INDUCTOR-RESCUE-fk-naturalist
- removed Q5: 2N7002LT1G, conservify:SOT-23, symbol RocketScreamKicadLibrary:MOSFET-N
- removed R101, R102, R103: 10K, conservify:RES-0603, symbol conservify:RESISTOR
- removed R26, R27: 4.7K, conservify:RES-0603, symbol conservify:RESISTOR
- removed R38, R44: 100K, conservify:RES-0603, symbol conservify:RESISTOR
- removed R45: 22K1, conservify:RES-0603, symbol conservify:RESISTOR
- removed U103: BNO055, conservify:BNO055, symbol fk-naturalist-rescue:BNO055-RESCUE-fk-naturalist
- removed U3: SK6812, conservify:SK6812, symbol conservify:SK6812
- removed U8: MCP1700T-3302E/MB, conservify:SOT-89, symbol conservify:MCP1700T-XXX2E
- removed U9: ISL8541x, conservify:DFN-12-1EP_3x4mm_Pitch0.5mm, symbol fk-naturalist-rescue:ISL8541x
- removed Y101: FC-135, conservify:ABS07, symbol conservify:CRYSTAL
- added C13, C15, C16, C33: 100nF, conservify:CAP-0603, symbol conservify:CAPACITOR_CERAMIC
- added C17, C34: 10uF, conservify:CAP-0603, symbol conservify:CAPACITOR_CERAMIC
- added C2: 47uF, conservify:CAP-0603, symbol conservify:CAPACITOR_CERAMIC
- added C21, C26: 1uF, conservify:CAP-0603, symbol conservify:CAPACITOR_CERAMIC
- added C23, C29: 470pF, conservify:CAP-0603, symbol conservify:CAPACITOR_CERAMIC
- added C25, C30: 2.2uF, conservify:CAP-0603, symbol conservify:CAPACITOR_CERAMIC
- added J1: RF-SMA-EDGE, conservify:RF-SMA-EDGE, symbol conservify:RF_SMA_EDGE
- added J12, J14, J2: Conn_01x02, conservify:SJ_OPEN, symbol conservify:CONN_01x02
- added J13: CONN_01x06, conservify:JST_SH_BM06B-SRSS-TB_1x06-1MP_P1.00mm_Vertical, symbol conservify:CONN_01x06
- added J3: S2B-PH-SM4-TB, conservify:S2B-PH-SM4-TB, symbol conservify:S2B_PH_SM4_TB
- added J4: Conn_01x01, conservify:Socket_Strip_Straight_1x01_Pitch2.54mm, symbol conservify:CONN_01x01
- added J5: CONN_01x03_SERIAL, conservify:Molex_CLIK-Mate_502382-0370_1x03_P1.25mm_Vertical, symbol conservify:CONN_01x03_SERIAL
- added J8: CONN_01x02, conservify:Molex_CLIK-Mate_502382-0270_1x02_P1.25mm_Vertical, symbol conservify:CONN_01x02
- added R11, R13: 100K, conservify:RES-0603, symbol conservify:RESISTOR
- added R12, R14: 165.7K, conservify:RES-0603, symbol conservify:RESISTOR
- added R7: 10K, conservify:RES-0603, symbol conservify:RESISTOR
- added U12: TPS2052B, conservify:SOIC-8-N, symbol conservify:TPS2052B
- added U13: SK6812, conservify:SK6812, symbol conservify:SK6812
- added U14: MCP1700T-3302E/MB, conservify:SOT-89, symbol conservify:MCP1700T-XXX2E
- added U3: RFM95W, conservify:RFM9xW, symbol conservify:RFM9xW
- added U8, U9: TL5209, conservify:SOIC-8-N, symbol conservify:TL5209
- BT1: symbol fk-naturalist-rescue:Battery_Cell -> conservify:BATTERY_CELL; MFN Harwin -> (none); MFP S8411-45R -> (none)
- C1, C10, C11, C12, C14, C18, C19, C20, C22, C24, C27, C28, C3, C4, C5, C6, C7, C8, C9: symbol RocketScreamKicadLibrary:CAPACITOR-CERAMIC -> conservify:CAPACITOR_CERAMIC
- D1, D10, D11, D2, D3, D9: symbol RocketScreamKicadLibrary:LED-SINGLE -> conservify:LED_SINGLE
- D7: symbol RocketScreamKicadLibrary:DIODE_DUAL_Schottky -> conservify:DIODE_DUAL_SCHOTTKY
- D8: symbol fk-naturalist-rescue:PRTR5V0U2X-RESCUE-fk-naturalist -> conservify:PRTR5V0U2X
- J10: symbol RocketScreamKicadLibrary:S2B-PH-SM4-TB -> conservify:S2B_PH_SM4_TB
- J11: symbol RocketScreamKicadLibrary:RF-SMA-EDGE -> conservify:RF_SMA_EDGE; MFP (none) -> S01-SJEDM-11BS05
- J6: symbol fk-naturalist-rescue:Conn_01x05 -> conservify:CONN_01x05
- J7: symbol RocketScreamKicadLibrary:CONN-HDR-2x5 -> conservify:CONN_02x05_SWD
- J9: symbol RocketScreamKicadLibrary:MICRO-USB -> conservify:MICRO_USB
- L1, L2: symbol fk-naturalist-rescue:INDUCTOR-RESCUE-fk-naturalist -> conservify:INDUCTOR
- M1, M3, M4, M6: footprint conservify:HOLE_NPTH_2.2MM -> conservify:HOLE_NPTH_2.54MM
- M10, M11, M2, M5, M8, M9: Critical (none) -> (none); MFN (none) -> (none); MFP (none) -> (none); Notes (none) -> (none); Package (none) -> (none); SPN1 (none) -> (none); Source (none) -> ANY; Subsystem (none) -> (none); Supplier1 (none) -> (none)
- M7: symbol fk-naturalist-rescue:MICROSD -> conservify:MICRO_SD
- Q1: symbol RocketScreamKicadLibrary:MOSFET-N -> conservify:MOSFET_N
- R23: SPN1 (none) -> 603-RC0603FR-07100KL; spn1 603-RC0603FR-07100KL -> (none)
- R37, R39, R4, R40, R5: MFN Yageo -> (none); MFP RC0603FR-071KL -> (none); spn1 603-RC0603FR-071KL -> 603-RC0603FR-07330RL
- SW1, SW2: symbol RocketScreamKicadLibrary:TACT-SWITCH_2Pins -> conservify:SWITCH_CONN_02
- U1: symbol fk-naturalist-rescue:ATWINC1500-MR210PA -> conservify:ATWINC1500_MR210PA
- U2: symbol RocketScreamKicadLibrary:ATSAMD21G18A-AU -> conservify:ATSAMD21G18A_AU
Connections:
- net labels added: A1_WIFI_RST, A2_WIFI_IRQ, A4_GPS_EN, D0_RADIO_D2, D12_SD_CS, D1_RADIO_D1, D26_FLASH_CS, D2_RADIO_D0, D2_WIFI_EN, D5_RADIO_CS, D6_USER_SW, D7_WIFI_CS, D8_WIFI_WAKE, D9_MODULE_EN, GPS_3V3, MODULE_3V3, PERIPH_3V3, PERIPH_EN
- net labels removed: A4, AREF, FLASH_CS, I2S_BCLK, I2S_DATA, I2S_WS, ISL_VIN, PERIPH_ENABLE, PERIPH_GND, RADIO_CS, RADIO_D0, RADIO_EN, RADIO_RST, SD_CS, USER_SW, WIFI_CS, WIFI_EN, WIFI_IRQ, WIFI_RST, WIFI_WAKE
- wire segments 516 -> 534
- no-connect marks 33 -> 42
Other:
- note added: "FIDUCIALS"
- note added: "LED"
- note removed: "BNO055"

Commit message: Add new 9 pin sensor connector.
Parts:
- removed J6: Conn_01x05, conservify:Molex_CLIK-Mate_502382-0570_1x05_P1.25mm_Vertical, symbol conservify:CONN_01x05
- added J6: CONN_01x09, conservify:Molex_CLIK-Mate_502382-0970_1x09_P1.25mm_Vertical, symbol conservify:CONN_01x09
Connections:
- net labels added: I2S_BCLK, I2S_DATA, I2S_WS
- net labels removed: A5
- wire segments 534 -> 538
- no-connect marks 42 -> 39
Changed lines of the file:
@@
 $EndComp
 $Comp
-L conservify:CONN_01x05 J6
-U 1 1 5A5962A1
-P 1550 9450
-F 0 "J6" H 1550 9750 50  0000 C CNN
-F 1 "Conn_01x05" H 1550 9150 50  0000 C CNN
-F 2 "conservify:Molex_CLIK-Mate_502382-0570_1x05_P1.25mm_Vertical" H 1550 9450 50  0001 C CNN
-F 3 "" H 1550 9450 50  0001 C CNN
-F 4 " " H 1550 9850 50  0001 C CNN "Critical"
-F 5 "Molex" H 1550 9850 50  0001 C CNN "MFN"
-F 6 "502382-0570" H 1550 9850 50  0001 C CNN "MFP"
-F 7 " " H 1550 9850 50  0001 C CNN "Notes"
-F 8 " " H 1550 9850 50  0001 C CNN "Package"
-F 9 "ANY" H 1550 9850 50  0001 C CNN "Source"
-F 10 " " H 1550 9850 50  0001 C CNN "Subsystem"
-F 11 "538-502382-0570" H 1550 9450 60  0001 C CNN "spn1"
-F 12 "mouser" H 1550 9450 60  0001 C CNN "supplier1"
-	1    1550 9450
-	1    0    0    -1
-$EndComp
-$Comp
 L conservify:GND #PWR065
 U 1 1 5A5962A2
-P 1100 9350
-F 0 "#PWR065" H 1100 9100 50  0001 C CNN
-F 1 "GND" H 1100 9200 50  0001 C CNN
-F 2 "" H 1100 9350 60  0000 C CNN
-F 3 "" H 1100 9350 60  0000 C CNN
-	1    1100 9350
-	0    1    1    0
+P 3000 9950
+F 0 "#PWR065" H 3000 9700 50  0001 C CNN
+F 1 "GND" H 3000 9800 50  0001 C CNN
+F 2 "" H 3000 9950 60  0000 C CNN
+F 3 "" H 3000 9950 60  0000 C CNN
+	1    3000 9950
+	0    -1   -1   0
 $EndComp
 $Comp
@@
 $EndComp
 $Comp
-L conservify:VBUS #PWR074
-U 1 1 5B28222B
-P 800 9450
-F 0 "#PWR074" H 800 9300 50  0001 C CNN
-F 1 "VBUS" H 800 9590 50  0000 C CNN
-F 2 "" H 800 9450 60  0000 C CNN
-F 3 "" H 800 9450 60  0000 C CNN
-	1    800  9450
-	1    0    0    -1
-$EndComp
-$Comp
 L conservify:FIDUCIAL M2
 U 1 1 5B2838D8
@@
 Text Label 4550 2900 0    50   ~ 0
 SCK
-Text Label 4550 3400 0    50   ~ 0
-A5
 Text Label 4550 4000 0    50   ~ 0
 USB+
@@
 Text Label 1100 10300 0    50   ~ 0
 D30
-Text Label 1200 9650 0    50   ~ 0
+Text Label 2850 9550 0    50   ~ 0
 SDA
-Text Label 1200 9550 0    50   ~ 0
+Text Label 2850 9450 0    50   ~ 0
 SCL
 Text Notes 13400 8650 0    180  ~ 36
@@
 Text Label 15700 14950 0    50   ~ 0
 D0_RADIO_D2
-Text Label 2000 3100 0    50   ~ 0
+Text Label 4850 3500 0    50   ~ 0
 D1_RADIO_D1
-Text Label 2000 3200 0    50   ~ 0
+Text Label 4850 3600 0    50   ~ 0
 D0_RADIO_D2
-Text Label 2000 2800 0    50   ~ 0
+Text Label 4550 3400 0    50   ~ 0
 D9_MODULE_EN
 Text Label 16650 3450 0    50   ~ 0
@@
 Text Label 20350 3350 0    60   ~ 0
 MODULE_3V3
-Text Label 800  9250 0    60   ~ 0
+Text Label 2850 9150 0    60   ~ 0
 MODULE_3V3
 Text Label 21500 3450 0    60   ~ 0
@@
 	1100 10300 1350 10300
 Wire Wire Line
-	1100 9350 1350 9350
-Wire Wire Line
-	1200 9550 1350 9550
-Wire Wire Line
-	1200 9650 1350 9650
-Wire Wire Line
 	12700 5600 12700 5800
 Wire Wire Line
@@
 	800  14300 1600 14300
 Wire Wire Line
-	1350 9450 800  9450
-Wire Wire Line
 	10950 6550 11050 6550
 Wire Wire Line
@@
 	20250 3350 20900 3350
 Wire Wire Line
-	800  9250 1350 9250
-Wire Wire Line
 	21500 3350 21800 3350
 Wire Wire Line
@@
 NoConn ~ 8700 1600
 NoConn ~ 16550 5650
-NoConn ~ 5100 3400
-NoConn ~ 2000 2900
-NoConn ~ 2000 3000
 $Comp
 L conservify:5V0 #PWR0115
@@
 Wire Wire Line
 	4550 2700 5100 2700
+$Comp
+L conservify:CONN_01x09 J6
+U 1 1 5B99BF77
+P 2600 9550
+F 0 "J6" H 2600 9050 50  0000 L CNN
+F 1 "CONN_01x09" V 2700 9350 50  0000 L CNN
+F 2 "conservify:Molex_CLIK-Mate_502382-0970_1x09_P1.25mm_Vertical" H 2600 9550 50  0001 C CNN
+F 3 "" H 2600 9550 50  0001 C CNN
+	1    2600 9550
+	-1   0    0    1
+$EndComp
+Text Label 2850 9250 0    50   ~ 0
+SCL2
+Text Label 2850 9350 0    50   ~ 0
+SDA2
+Text Label 2850 9650 0    50   ~ 0
+I2S_DATA
+Text Label 2850 9750 0    50   ~ 0
+I2S_WS
+Text Label 2850 9850 0    50   ~ 0
+I2S_BCLK
+Wire Wire Line
+	2800 9150 3450 9150
+Wire Wire Line
+	3450 9250 2800 9250
+Wire Wire Line
+	2800 9350 3450 9350
+Wire Wire Line
+	3450 9450 2800 9450
+Wire Wire Line
+	2800 9550 3450 9550
+Wire Wire Line
+	3450 9650 2800 9650
+Wire Wire Line
+	2800 9750 3450 9750
+Wire Wire Line
+	3450 9850 2800 9850
+Wire Wire Line
+	2800 9950 3000 9950
+Text Label 2000 2800 0    50   ~ 0
+I2S_DATA
+Text Label 2000 3200 0    50   ~ 0
+I2S_WS
+Text Label 2000 3100 0    50   ~ 0
+I2S_BCLK
 $EndSCHEMATC

Commit message: Use more compatible FP for flash.
Parts:
- U5: footprint conservify:SOIC-8-N -> conservify:SOIC-8-N-WIDE
Connections:
- wire segments 538 -> 541
Changed lines of the file:
@@
 F 0 "U5" H 10150 9650 60  0000 C CNN
 F 1 "S25FL116K0XMFI041" H 10150 9050 60  0000 C CNN
-F 2 "conservify:SOIC-8-N" H 10150 8950 60  0001 C CNN
+F 2 "conservify:SOIC-8-N-WIDE" H 10150 8950 60  0001 C CNN
 F 3 "" H 9950 9400 60  0000 C CNN
 F 4 " " H 10150 9750 50  0001 C CNN "Critical"
@@
 U 1 1 5A596200
 P 11750 3300
-F 0 "R34" V 11750 3150 60  0000 C CNN
-F 1 "10K" V 11850 3150 60  0000 C CNN
+F 0 "R34" V 11700 3150 60  0000 C CNN
+F 1 "10K" V 11800 3150 60  0000 C CNN
 F 2 "conservify:RES-0603" H 11750 3100 60  0001 C CNN
 F 3 "" H 11750 3300 60  0000 C CNN
@@
 U 1 1 5A596202
 P 12050 3000
-F 0 "C19" H 12100 3100 50  0000 L CNN
-F 1 "4.7uF" V 11900 2650 50  0000 L CNN
+F 0 "C19" V 12100 2800 50  0000 L CNN
+F 1 "4.7uF" V 11950 2750 50  0000 L CNN
 F 2 "conservify:CAP-0603" H 12050 2800 30  0001 C CNN
 F 3 "" H 12050 3000 60  0000 C CNN
@@
 U 1 1 5A596248
 P 18850 9550
-F 0 "C27" H 18900 9650 50  0000 L CNN
-F 1 "1uF" V 18700 9200 50  0000 L CNN
+F 0 "C27" V 18750 9600 50  0000 L CNN
+F 1 "1uF" V 18750 9350 50  0000 L CNN
 F 2 "conservify:CAP-0603" H 18850 9350 30  0001 C CNN
 F 3 "" H 18850 9550 60  0000 C CNN
@@
 L conservify:RESISTOR R41
 U 1 1 5A59624A
-P 18850 9250
-F 0 "R41" H 18725 9350 60  0000 C CNN
-F 1 "180R" H 18950 9350 60  0000 C CNN
-F 2 "conservify:RES-0603" H 18850 9050 60  0001 C CNN
-F 3 "" H 18850 9250 60  0000 C CNN
-F 4 " " H 18725 9450 50  0001 C CNN "Critical"
-F 5 "Yageo" H 18725 9450 50  0001 C CNN "MFN"
-F 6 "RC0603FR-07180RL" H 18725 9450 50  0001 C CNN "MFP"
-F 7 " " H 18725 9450 50  0001 C CNN "Notes"
-F 8 " " H 18725 9450 50  0001 C CNN "Package"
-F 9 "ANY" H 18725 9450 50  0001 C CNN "Source"
-F 10 " " H 18725 9450 50  0001 C CNN "Subsystem"
-F 11 "0.1" H 18725 9450 50  0001 C CNN "price"
-F 12 "603-RC0603FR-07180RL" H 18825 9450 50  0001 C CNN "spn1"
-F 13 "mouser" H 5400 5050 50  0001 C CNN "supplier1"
-	1    18850 9250
+P 18450 9250
+F 0 "R41" H 18325 9350 60  0000 C CNN
+F 1 "180R" H 18550 9350 60  0000 C CNN
+F 2 "conservify:RES-0603" H 18450 9050 60  0001 C CNN
+F 3 "" H 18450 9250 60  0000 C CNN
+F 4 " " H 18325 9450 50  0001 C CNN "Critical"
+F 5 "Yageo" H 18325 9450 50  0001 C CNN "MFN"
+F 6 "RC0603FR-07180RL" H 18325 9450 50  0001 C CNN "MFP"
+F 7 " " H 18325 9450 50  0001 C CNN "Notes"
+F 8 " " H 18325 9450 50  0001 C CNN "Package"
+F 9 "ANY" H 18325 9450 50  0001 C CNN "Source"
+F 10 " " H 18325 9450 50  0001 C CNN "Subsystem"
+F 11 "0.1" H 18325 9450 50  0001 C CNN "price"
+F 12 "603-RC0603FR-07180RL" H 18425 9450 50  0001 C CNN "spn1"
+F 13 "mouser" H 5000 5050 50  0001 C CNN "supplier1"
+	1    18450 9250
 	1    0    0    -1
 $EndComp
@@
 U 1 1 5A59624B
 P 18100 9350
-F 0 "R40" H 17975 9450 60  0000 C CNN
-F 1 "1K" H 18200 9450 60  0000 C CNN
+F 0 "R40" H 17900 9300 60  0000 C CNN
+F 1 "1K" H 18300 9300 60  0000 C CNN
 F 2 "conservify:RES-0603" H 18100 9150 60  0001 C CNN
 F 3 "" H 18100 9350 60  0000 C CNN
@@
 L conservify:3V3 #PWR048
 U 1 1 5A59624D
-P 18400 9200
-F 0 "#PWR048" H 18400 9050 50  0001 C CNN
-F 1 "3V3" H 18400 9340 50  0000 C CNN
-F 2 "" H 18400 9200 60  0000 C CNN
-F 3 "" H 18400 9200 60  0000 C CNN
-	1    18400 9200
+P 17850 9250
+F 0 "#PWR048" H 17850 9100 50  0001 C CNN
+F 1 "3V3" H 17850 9390 50  0000 C CNN
+F 2 "" H 17850 9250 60  0000 C CNN
+F 3 "" H 17850 9250 60  0000 C CNN
+	1    17850 9250
 	1    0    0    -1
 $EndComp
@@
 L conservify:CAPACITOR_CERAMIC C28
 U 1 1 5A59625D
-P 19200 8950
-F 0 "C28" H 19250 9050 50  0000 L CNN
-F 1 "10nF" V 19050 8950 50  0000 L CNN
-F 2 "conservify:CAP-0603" H 19200 8750 30  0001 C CNN
-F 3 "" H 19200 8950 60  0000 C CNN
-F 4 " " H 19250 9150 50  0001 C CNN "Critical"
-F 5 "AVX" H 19250 9150 50  0001 C CNN "MFN"
-F 6 "0603YC103K4T2A" H 19250 9150 50  0001 C CNN "MFP"
-F 7 " " H 19250 9150 50  0001 C CNN "Notes"
-F 8 " " H 19250 9150 50  0001 C CNN "Package"
-F 9 "ANY" H 19250 9150 50  0001 C CNN "Source"
-F 10 " " H 19250 9150 50  0001 C CNN "Subsystem"
-F 11 "0.4" H 19250 9150 50  0001 C CNN "price"
-F 12 "581-0603YC103K4T2A" H 5750 4450 50  0001 C CNN "spn1"
-F 13 "mouser" H 5750 4450 50  0001 C CNN "supplier1"
-	1    19200 8950
+P 18850 8950
+F 0 "C28" H 18900 9050 50  0000 L CNN
+F 1 "10nF" V 18750 9000 50  0000 L CNN
+F 2 "conservify:CAP-0603" H 18850 8750 30  0001 C CNN
+F 3 "" H 18850 8950 60  0000 C CNN
+F 4 " " H 18900 9150 50  0001 C CNN "Critical"
+F 5 "AVX" H 18900 9150 50  0001 C CNN "MFN"
+F 6 "0603YC103K4T2A" H 18900 9150 50  0001 C CNN "MFP"
+F 7 " " H 18900 9150 50  0001 C CNN "Notes"
+F 8 " " H 18900 9150 50  0001 C CNN "Package"
+F 9 "ANY" H 18900 9150 50  0001 C CNN "Source"
+F 10 " " H 18900 9150 50  0001 C CNN "Subsystem"
+F 11 "0.4" H 18900 9150 50  0001 C CNN "price"
+F 12 "581-0603YC103K4T2A" H 5400 4450 50  0001 C CNN "spn1"
+F 13 "mouser" H 5400 4450 50  0001 C CNN "supplier1"
+	1    18850 8950
 	1    0    0    -1
 $EndComp
@@
 L conservify:GND #PWR053
 U 1 1 5A59625E
-P 19400 8700
-F 0 "#PWR053" H 19400 8450 50  0001 C CNN
-F 1 "GND" H 19400 8550 50  0001 C CNN
-F 2 "" H 19400 8700 60  0000 C CNN
-F 3 "" H 19400 8700 60  0000 C CNN
-	1    19400 8700
+P 19000 8700
+F 0 "#PWR053" H 19000 8450 50  0001 C CNN
+F 1 "GND" H 19000 8550 50  0001 C CNN
+F 2 "" H 19000 8700 60  0000 C CNN
+F 3 "" H 19000 8700 60  0000 C CNN
+	1    19000 8700
 	0    -1   -1   0
 $EndComp
@@
 U 1 1 5A59627C
 P 12200 1700
-F 0 "D9" V 12250 1500 50  0000 C CNN
-F 1 "Green" V 12150 1500 50  0000 C CNN
+F 0 "D9" H 12350 1650 50  0000 C CNN
+F 1 "Green" H 12200 1800 50  0000 C CNN
 F 2 "conservify:LED-0603" H 12200 1450 60  0001 C CNN
 F 3 "" H 12200 1700 60  0000 C CNN
@@
 U 1 1 5A59627D
 P 12200 1900
-F 0 "D10" V 12250 1700 50  0000 C CNN
-F 1 "Red" V 12150 1700 50  0000 C CNN
+F 0 "D10" H 12350 1850 50  0000 C CNN
+F 1 "Red" H 12200 1750 50  0000 C CNN
 F 2 "conservify:LED-0603" H 12200 1650 60  0001 C CNN
 F 3 "" H 12200 1900 60  0000 C CNN
@@
 	18850 9700 18850 9750
 Wire Wire Line
-	19100 9250 19200 9250
+	18700 9250 18850 9250
 Wire Wire Line
 	17850 9350 17500 9350
 Wire Wire Line
-	18400 9200 18400 9250
-Wire Wire Line
-	18400 9250 18600 9250
-Wire Wire Line
 	20800 9250 21050 9250
 Wire Wire Line
@@
 	2000 3800 2850 3800
 Wire Wire Line
-	19200 9250 19200 9100
+	18850 9250 18850 9100
 Wire Wire Line
-	19400 8700 19200 8700
+	19000 8700 18850 8700
 Wire Wire Line
-	19200 8700 19200 8800
+	18850 8700 18850 8800
 Wire Wire Line
 	1600 14200 1600 14300
@@
 	19150 9550 19150 9650
 Wire Wire Line
-	18850 9350 19300 9350
-Wire Wire Line
 	21350 7550 21350 7650
 Wire Wire Line
@@
 	5450 14200 5450 14300
 Wire Wire Line
-	19200 9250 19300 9250
+	18850 9250 19250 9250
 Wire Wire Line
 	4450 15300 4450 15400
@@
 Connection ~ 5450 14300
 Connection ~ 5450 14200
-Connection ~ 19200 9250
+Connection ~ 18850 9250
 Connection ~ 4450 15300
 Connection ~ 4400 12300
@@
 Text Label 2000 3100 0    50   ~ 0
 I2S_BCLK
+$Comp
+L conservify:PWR_FLAG #FLG0101
+U 1 1 5B8B284F
+P 19250 9100
+F 0 "#FLG0101" H 19250 9175 50  0001 C CNN
+F 1 "PWR_FLAG" V 19300 9200 50  0000 C CNN
+F 2 "" H 19250 9100 50  0001 C CNN
+F 3 "~" H 19250 9100 50  0001 C CNN
+	1    19250 9100
+	1    0    0    -1
+$EndComp
+Wire Wire Line
+	17850 9250 18200 9250
+Wire Wire Line
+	19250 9100 19250 9250
+Connection ~ 19250 9250
+Wire Wire Line
+	19250 9250 19300 9250
+$Comp
+L conservify:PWR_FLAG #FLG0108
+U 1 1 5BB1F2A5
+P 19050 9550
+F 0 "#FLG0108" H 19050 9625 50  0001 C CNN
+F 1 "PWR_FLAG" V 19100 9600 50  0000 C CNN
+F 2 "" H 19050 9550 50  0001 C CNN
+F 3 "~" H 19050 9550 50  0001 C CNN
+	1    19050 9550
+	-1   0    0    1
+$EndComp
+Wire Wire Line
+	18850 9350 19050 9350
+Wire Wire Line
+	19050 9350 19050 9550
+Connection ~ 19050 9350
+Wire Wire Line
+	19050 9350 19300 9350
 $EndSCHEMATC

Commit message: Consistency in part values
Parts:
- J12, J14, J2: value Conn_01x02 -> CONN_01x02
- J6: Critical (none) -> (none); MFN (none) -> Molex; MFP (none) -> 502382-0970; Notes (none) -> (none); Package (none) -> (none); SPN1 (none) -> WM4786CT-ND; Source (none) -> ANY; Subsystem (none) -> (none); Supplier1 (none) -> digikey

Commit message: Fix SD landing.
Parts:
- M7: value MICROSD -> MICRO-SD; footprint conservify:MICROSD -> conservify:MICRO-SD
Changed lines of the file:
@@
 P 6400 13500
 F 0 "M7" H 6400 13500 45 0001 C CNN
-F 1 "MICROSD" H 6400 13500 45 0001 C CNN
-F 2 "conservify:MICROSD" H 6430 13650 20 0001 C CNN
+F 1 "MICRO-SD" H 6400 13500 45 0001 C CNN
+F 2 "conservify:MICRO-SD" H 6430 13650 20 0001 C CNN
 F 3 "" H 6400 13500 60 0001 C CNN
 F 4 " " H 6400 13600 50 0001 C CNN "Critical"
