File: hardware/main-board/fk-naturalist.sch (KiCad schematic (older format))
At the start: 121 parts, among them J1 RF-SMA-EDGE, J10 S2B-PH-SM4-TB, J11 RF-SMA-EDGE, J12 CONN_01x02, J13 CONN_01x06, J14 CONN_01x02, J2 CONN_01x02, J3 S2B-PH-SM4-TB, J4 Conn_01x01, J5 CONN_01x03_SERIAL, J6 CONN_01x09, J7 CONN_02x05_SWD, J8 CONN_01x02, J9 MICRO-USB, M1 MOUNT_HOLE, M10 FIDUCIAL, M11 FIDUCIAL, M2 FIDUCIAL, M3 MOUNT_HOLE, M4 MOUNT_HOLE, M5 FIDUCIAL, M6 MOUNT_HOLE, M7 MICRO-SD, M8 FIDUCIAL, M9 FIDUCIAL, Q1 2N7002LT1G, SW1 SPNO, SW2 SPNO, U1 ATWINC1500-MR210PA, U10 FGPMMOPA6H, U11 MAX1704XX, U12 TPS2052B, U13 SK6812, U14 MCP1700T-3302E/MB, U2 ATSAMD21G18A-AU, U3 RFM95W, U4 24AA02E64, U5 S25FL116K0XMFI041, U6 BQ24074RGTT, U7 PCF8523, U8 TL5209, U9 TL5209, Y1 FC-135, Y2 FC-135

Commit message: Add some bypass caps on GPS 3v3, see if fix issues are power related.
Parts:
- added C31: 10uF, conservify:CAP-0603, symbol conservify:CAPACITOR_CERAMIC
- added C32: 47uF, conservify:CAP-0603, symbol conservify:CAPACITOR_CERAMIC
- added C35: 100nF, conservify:CAP-0603, symbol conservify:CAPACITOR_CERAMIC
Connections:
- wire segments 541 -> 550
- no-connect marks 39 -> 38

Commit message: Add a bead on the GPS 3v3 supply too.
Parts:
- added L3: BLM18KG221SN1D, conservify:IND-0603, symbol conservify:INDUCTOR
Connections:
- wire segments 550 -> 554
Changed lines of the file:
@@
 L conservify:CONN_01x06 J13
 U 1 1 5B6988D1
-P 16350 5950
-F 0 "J13" H 16270 5425 50  0000 C CNN
-F 1 "CONN_01x06" H 16270 5516 50  0000 C CNN
-F 2 "conservify:JST_SH_BM06B-SRSS-TB_1x06-1MP_P1.00mm_Vertical" H 16350 5950 50  0001 C CNN
-F 3 "" H 16350 5950 50  0001 C CNN
-F 4 " " H 16270 5525 50  0001 C CNN "Critical"
-F 5 "JST" H 16270 5525 50  0001 C CNN "MFN"
-F 6 "BM06B-SRSS-TB(LF)(SN)" H 16270 5525 50  0001 C CNN "MFP"
-F 7 " " H 16270 5525 50  0001 C CNN "Notes"
-F 8 " " H 16270 5525 50  0001 C CNN "Package"
-F 9 "455-1792-1-ND" H 16270 5525 50  0001 C CNN "SPN1"
-F 10 "ANY" H 16270 5525 50  0001 C CNN "Source"
-F 11 " " H 16270 5525 50  0001 C CNN "Subsystem"
-F 12 "digikey" H 16270 5525 50  0001 C CNN "Supplier1"
-	1    16350 5950
-	-1   0    0    1
+P 22450 6000
+F 0 "J13" H 22370 5475 50  0000 C CNN
+F 1 "CONN_01x06" H 22370 5566 50  0000 C CNN
+F 2 "conservify:JST_SH_BM06B-SRSS-TB_1x06-1MP_P1.00mm_Vertical" H 22450 6000 50  0001 C CNN
+F 3 "" H 22450 6000 50  0001 C CNN
+F 4 " " H 22370 5575 50  0001 C CNN "Critical"
+F 5 "JST" H 22370 5575 50  0001 C CNN "MFN"
+F 6 "BM06B-SRSS-TB(LF)(SN)" H 22370 5575 50  0001 C CNN "MFP"
+F 7 " " H 22370 5575 50  0001 C CNN "Notes"
+F 8 " " H 22370 5575 50  0001 C CNN "Package"
+F 9 "455-1792-1-ND" H 22370 5575 50  0001 C CNN "SPN1"
+F 10 "ANY" H 22370 5575 50  0001 C CNN "Source"
+F 11 " " H 22370 5575 50  0001 C CNN "Subsystem"
+F 12 "digikey" H 22370 5575 50  0001 C CNN "Supplier1"
+	1    22450 6000
+	1    0    0    -1
 $EndComp
 $Comp
 L conservify:GND #PWR0101
 U 1 1 5B699CD3
-P 17200 6200
-F 0 "#PWR0101" H 17200 5950 50  0001 C CNN
-F 1 "GND" H 17200 6050 50  0001 C CNN
-F 2 "" H 17200 6200 60  0000 C CNN
-F 3 "" H 17200 6200 60  0000 C CNN
-	1    17200 6200
-	1    0    0    -1
+P 21600 5750
+F 0 "#PWR0101" H 21600 5500 50  0001 C CNN
+F 1 "GND" H 21600 5600 50  0001 C CNN
+F 2 "" H 21600 5750 60  0000 C CNN
+F 3 "" H 21600 5750 60  0000 C CNN
+	1    21600 5750
+	-1   0    0    1
 $EndComp
 $Comp
@@
 Text Notes 8700 13500 0    180  ~ 36
 PERIPHERALS
-Text Label 18200 6150 0    60   ~ 0
+Text Label 16450 6150 0    60   ~ 0
 GPS_3V3
-Text Label 16600 6050 0    60   ~ 0
-GPS_3V3
-Text Label 16600 5850 0    50   ~ 0
+Text Label 22200 6100 2    50   ~ 0
 GPS_TX
-Text Label 16600 5950 0    50   ~ 0
+Text Label 22200 6000 2    50   ~ 0
 GPS_RX
-Text Label 16600 5750 0    60   ~ 0
+Text Label 22200 6200 2    60   ~ 0
 BAT_BACKUP
 Text Label 15700 14850 0    50   ~ 0
@@
 	1600 12900 1600 13700
 Wire Wire Line
-	16550 5750 17200 5750
-Wire Wire Line
-	17200 5850 16550 5850
-Wire Wire Line
-	17200 5950 16550 5950
-Wire Wire Line
-	16550 6050 17200 6050
-Wire Wire Line
-	17200 6150 16550 6150
-Wire Wire Line
-	17200 6200 17200 6150
+	22250 6200 21600 6200
+Wire Wire Line
+	21600 6100 22250 6100
+Wire Wire Line
+	21600 6000 22250 6000
+Wire Wire Line
+	21600 5800 22250 5800
+Wire Wire Line
+	21600 5750 21600 5800
 Wire Wire Line
 	15700 14850 16250 14850
@@
 NoConn ~ 8700 1000
 NoConn ~ 8700 1600
-NoConn ~ 16550 5650
+NoConn ~ 22250 6300
 NoConn ~ 4100 7450
 NoConn ~ 3650 7450
@@
 	17900 5950 17900 6150
 Wire Wire Line
-	17900 6150 18900 6150
+	17900 6150 18600 6150
 Wire Wire Line
 	17550 5650 17550 5500
@@
 Wire Wire Line
 	17900 5350 17900 5500
+$Comp
+L conservify:INDUCTOR L3
+U 1 1 5B980CDB
+P 17250 6150
+F 0 "L3" H 17250 6100 50  0000 C CNN
+F 1 "BLM18KG221SN1D" H 17250 6250 50  0000 C CNN
+F 2 "conservify:IND-0603" H 17250 6000 60  0001 C CNN
+F 3 "" V 17250 6150 60  0000 C CNN
+F 4 " " H 17250 6200 50  0001 C CNN "Critical"
+F 5 "Murata Electronics" H 17250 6200 50  0001 C CNN "MFN"
+F 6 "BLM18KG221SN1D" H 17250 6200 50  0001 C CNN "MFP"
+F 7 " " H 17250 6200 50  0001 C CNN "Notes"
+F 8 " " H 17250 6200 50  0001 C CNN "Package"
+F 9 "ANY" H 17250 6200 50  0001 C CNN "Source"
+F 10 " " H 17250 6200 50  0001 C CNN "Subsystem"
+F 11 "0.1" H 17250 6200 50  0001 C CNN "price"
+F 12 "81-BLM18KG221SN1D" H 9350 -100 50  0001 C CNN "spn1"
+F 13 "mouser" H 9350 -100 50  0001 C CNN "supplier1"
+	1    17250 6150
+	1    0    0    -1
+$EndComp
+Wire Wire Line
+	16450 6150 16950 6150
+Wire Wire Line
+	17550 6150 17900 6150
+Connection ~ 17900 6150
+Wire Wire Line
+	18600 6150 18600 5900
+Wire Wire Line
+	18600 5900 22250 5900
+Connection ~ 18600 6150
+Wire Wire Line
+	18600 6150 18900 6150
 $EndSCHEMATC

Commit message: Fix Rx/Tx on backup GPS.
Changed lines of the file:
@@
 Text Label 16450 6150 0    60   ~ 0
 GPS_3V3
-Text Label 22200 6100 2    50   ~ 0
+Text Label 21950 6000 2    50   ~ 0
 GPS_TX
-Text Label 22200 6000 2    50   ~ 0
+Text Label 21950 6100 2    50   ~ 0
 GPS_RX
 Text Label 22200 6200 2    60   ~ 0

Commit message: Naturalist module enable pin is A5, D9 is used for I2S.
Connections:
- net labels added: A5_MODULE_EN
Changed lines of the file:
@@
 D0_RADIO_D2
 Text Label 4550 3400 0    50   ~ 0
-D9_MODULE_EN
+A5_MODULE_EN
 Text Label 16650 3450 0    50   ~ 0
 D9_MODULE_EN
