File: hardware/sensor-board/fk-naturalist-sensors.sch (KiCad schematic (older format))
At the start: 24 parts, among them J1 Conn_01x07, M1 MOUNT_HOLE, M10 FIDUCIAL, M2 MOUNT_HOLE, M3 MOUNT_HOLE, M4 MOUNT_HOLE, M5 FIDUCIAL, M6 FIDUCIAL, M7 FIDUCIAL, M8 FIDUCIAL, M9 FIDUCIAL, U1 MPL3115A2, U2 SHT31, U3 SPH0645, U4 TSL2591

Commit message: Move to footprints in our library.
Parts:
- C1, C2, C3, C4, C5, C6, C7: footprint RocketScreamKicadLibrary:CAP-0603 -> conservify:CAP-0603
- M10, M5, M6, M7, M8, M9: footprint Fiducials:Fiducial_0.75mm_Dia_1.5mm_Outer -> conservify:FIDUCIAL-1MM
- R1, R2: footprint RocketScreamKicadLibrary:RES-0603 -> conservify:RES-0603
Changed lines of the file:
@@
 F 0 "C1" V 4450 4350 50  0000 L CNN
 F 1 "100nF" V 4750 4300 50  0000 L CNN
-F 2 "RocketScreamKicadLibrary:CAP-0603" H 4600 4200 30  0001 C CNN
+F 2 "conservify:CAP-0603" H 4600 4200 30  0001 C CNN
 F 3 "" H 4600 4400 60  0000 C CNN
 F 4 "0" H 4450 4450 50  0001 C CNN "price"
@@
 F 0 "C3" V 4900 4350 50  0000 L CNN
 F 1 "100nF" V 5200 4300 50  0000 L CNN
-F 2 "RocketScreamKicadLibrary:CAP-0603" H 5050 4200 30  0001 C CNN
+F 2 "conservify:CAP-0603" H 5050 4200 30  0001 C CNN
 F 3 "" H 5050 4400 60  0000 C CNN
 F 4 "0" H 4900 4450 50  0001 C CNN "price"
@@
 F 0 "C5" V 5350 4350 50  0000 L CNN
 F 1 "10uF" V 5650 4300 50  0000 L CNN
-F 2 "RocketScreamKicadLibrary:CAP-0603" H 5500 4200 30  0001 C CNN
+F 2 "conservify:CAP-0603" H 5500 4200 30  0001 C CNN
 F 3 "" H 5500 4400 60  0000 C CNN
 F 4 "0" H 5350 4450 50  0001 C CNN "price"
@@
 F 0 "C4" V 5100 5950 50  0000 L CNN
 F 1 "1uF" V 5400 5950 50  0000 L CNN
-F 2 "RocketScreamKicadLibrary:CAP-0603" H 5250 5800 30  0001 C CNN
+F 2 "conservify:CAP-0603" H 5250 5800 30  0001 C CNN
 F 3 "" H 5250 6000 60  0000 C CNN
 F 4 "0" H 5100 6050 50  0001 C CNN "price"
@@
 F 0 "C2" V 4800 2700 50  0000 L CNN
 F 1 "100nF" V 5100 2650 50  0000 L CNN
-F 2 "RocketScreamKicadLibrary:CAP-0603" H 4950 2550 30  0001 C CNN
+F 2 "conservify:CAP-0603" H 4950 2550 30  0001 C CNN
 F 3 "" H 4950 2750 60  0000 C CNN
 F 4 "0" H 4800 2800 50  0001 C CNN "price"
@@
 F 0 "R1" H 2250 1350 60  0000 C CNN
 F 1 "10K" H 2250 1150 60  0000 C CNN
-F 2 "RocketScreamKicadLibrary:RES-0603" H 2250 1050 60  0001 C CNN
+F 2 "conservify:RES-0603" H 2250 1050 60  0001 C CNN
 F 3 "" H 2250 1250 60  0000 C CNN
 F 4 "0" H 2200 1150 50  0001 C CNN "price"
@@
 F 0 "R2" H 4750 1450 60  0000 C CNN
 F 1 "68R" H 4750 1250 60  0000 C CNN
-F 2 "RocketScreamKicadLibrary:RES-0603" H 4750 1150 60  0001 C CNN
+F 2 "conservify:RES-0603" H 4750 1150 60  0001 C CNN
 F 3 "" H 4750 1350 60  0000 C CNN
 F 4 "0" H 4700 1250 50  0001 C CNN "price"
@@
 F 0 "C7" V 6100 1250 50  0000 L CNN
 F 1 "220pF" V 6400 1250 50  0000 L CNN
-F 2 "RocketScreamKicadLibrary:CAP-0603" H 6250 1100 30  0001 C CNN
+F 2 "conservify:CAP-0603" H 6250 1100 30  0001 C CNN
 F 3 "" H 6250 1300 60  0000 C CNN
 F 4 "0" H 6100 1350 50  0001 C CNN "price"
@@
 F 0 "C6" V 5700 1250 50  0000 L CNN
 F 1 "1uF" V 6000 1250 50  0000 L CNN
-F 2 "RocketScreamKicadLibrary:CAP-0603" H 5850 1100 30  0001 C CNN
+F 2 "conservify:CAP-0603" H 5850 1100 30  0001 C CNN
 F 3 "" H 5850 1300 60  0000 C CNN
 F 4 "0" H 5700 1350 50  0001 C CNN "price"
@@
 F 0 "M5" H 7200 2500 60  0000 C CNN
 F 1 "FIDUCIAL" H 7200 2125 60  0000 C CNN
-F 2 "Fiducials:Fiducial_0.75mm_Dia_1.5mm_Outer" H 7200 2050 60  0001 C CNN
+F 2 "conservify:FIDUCIAL-1MM" H 7200 2050 60  0001 C CNN
 F 3 "" H 7200 2350 60  0000 C CNN
 	1    7200 2350
@@
 F 0 "M6" H 7700 2500 60  0000 C CNN
 F 1 "FIDUCIAL" H 7700 2125 60  0000 C CNN
-F 2 "Fiducials:Fiducial_0.75mm_Dia_1.5mm_Outer" H 7700 2050 60  0001 C CNN
+F 2 "conservify:FIDUCIAL-1MM" H 7700 2050 60  0001 C CNN
 F 3 "" H 7700 2350 60  0000 C CNN
 	1    7700 2350
@@
 F 0 "M7" H 8200 2500 60  0000 C CNN
 F 1 "FIDUCIAL" H 8200 2125 60  0000 C CNN
-F 2 "Fiducials:Fiducial_0.75mm_Dia_1.5mm_Outer" H 8200 2050 60  0001 C CNN
+F 2 "conservify:FIDUCIAL-1MM" H 8200 2050 60  0001 C CNN
 F 3 "" H 8200 2350 60  0000 C CNN
 	1    8200 2350
@@
 F 0 "M8" H 7200 3050 60  0000 C CNN
 F 1 "FIDUCIAL" H 7200 2675 60  0000 C CNN
-F 2 "Fiducials:Fiducial_0.75mm_Dia_1.5mm_Outer" H 7200 2600 60  0001 C CNN
+F 2 "conservify:FIDUCIAL-1MM" H 7200 2600 60  0001 C CNN
 F 3 "" H 7200 2900 60  0000 C CNN
 	1    7200 2900
@@
 F 0 "M9" H 7700 3050 60  0000 C CNN
 F 1 "FIDUCIAL" H 7700 2675 60  0000 C CNN
-F 2 "Fiducials:Fiducial_0.75mm_Dia_1.5mm_Outer" H 7700 2600 60  0001 C CNN
+F 2 "conservify:FIDUCIAL-1MM" H 7700 2600 60  0001 C CNN
 F 3 "" H 7700 2900 60  0000 C CNN
 	1    7700 2900
@@
 F 0 "M10" H 8200 3050 60  0000 C CNN
 F 1 "FIDUCIAL" H 8200 2675 60  0000 C CNN
-F 2 "Fiducials:Fiducial_0.75mm_Dia_1.5mm_Outer" H 8200 2600 60  0001 C CNN
+F 2 "conservify:FIDUCIAL-1MM" H 8200 2600 60  0001 C CNN
 F 3 "" H 8200 2900 60  0000 C CNN
 	1    8200 2900

Commit message: Fix DRC checks and rescued parts.
Parts:
- C1, C2, C3, C4, C5: symbol fk-naturalist-sensors-rescue:CAPACITOR-CERAMIC -> conservify:CAPACITOR_CERAMIC
Connections:
- wire segments 68 -> 70
- no-connect marks 4 -> 10
Changed lines of the file:
@@
 $EndComp
 $Comp
-L power1:GND #PWR01
+L conservify:GND #PWR01
 U 1 1 5B217CDE
 P 5050 4900
@@
 $EndComp
 $Comp
-L fk-naturalist-sensors-rescue:CAPACITOR-CERAMIC C1
+L conservify:CAPACITOR_CERAMIC C1
 U 1 1 5B217CDF
 P 4600 4400
@@
 $EndComp
 $Comp
-L fk-naturalist-sensors-rescue:CAPACITOR-CERAMIC C3
+L conservify:CAPACITOR_CERAMIC C3
 U 1 1 5B217CE0
 P 5050 4400
@@
 $EndComp
 $Comp
-L fk-naturalist-sensors-rescue:CAPACITOR-CERAMIC C5
+L conservify:CAPACITOR_CERAMIC C5
 U 1 1 5B217CE1
 P 5500 4400
@@
 $EndComp
 $Comp
-L power1:GND #PWR03
+L conservify:GND #PWR03
 U 1 1 5B217CE4
 P 5250 6350
@@
 $EndComp
 $Comp
-L fk-naturalist-sensors-rescue:CAPACITOR-CERAMIC C4
+L conservify:CAPACITOR_CERAMIC C4
 U 1 1 5B217CE6
 P 5250 6000
@@
 $EndComp
 $Comp
-L fk-naturalist-sensors-rescue:CAPACITOR-CERAMIC C2
+L conservify:CAPACITOR_CERAMIC C2
 U 1 1 5B217CE8
 P 4950 2750
@@
 $EndComp
 $Comp
-L power1:GND #PWR05
+L conservify:GND #PWR05
 U 1 1 5B217CE9
 P 4950 3050
@@
 $EndComp
 $Comp
-L power1:GND #PWR07
+L conservify:GND #PWR07
 U 1 1 5B217CFE
 P 2450 3050
@@
 $EndComp
 $Comp
-L power1:GND #PWR08
+L conservify:GND #PWR08
 U 1 1 5B217DC2
 P 1800 1650
@@
 $EndComp
 $Comp
-L power1:GND #PWR010
+L conservify:GND #PWR010
 U 1 1 5B217DC6
 P 6250 1550
@@
 $EndComp
 $Comp
-L power1:GND #PWR012
+L conservify:GND #PWR012
 U 1 1 5B21D250
 P 8300 4900
@@
 Wire Wire Line
 	5850 1150 6250 1150
+NoConn ~ 8200 2500
+NoConn ~ 7700 2500
+NoConn ~ 7200 2500
+NoConn ~ 7200 3050
+NoConn ~ 7700 3050
+NoConn ~ 8200 3050
+$Comp
+L conservify:3V3 #PWR0101
+U 1 1 5DA3D54E
+P 7200 5700
+F 0 "#PWR0101" H 7200 5550 50  0001 C CNN
+F 1 "3V3" H 7200 5840 50  0000 C CNN
+F 2 "" H 7200 5700 60  0000 C CNN
+F 3 "" H 7200 5700 60  0000 C CNN
+	1    7200 5700
+	1    0    0    -1
+$EndComp
+$Comp
+L conservify:GND #PWR0102
+U 1 1 5DA3D721
+P 7600 5700
+F 0 "#PWR0102" H 7600 5450 50  0001 C CNN
+F 1 "GND" H 7600 5550 50  0001 C CNN
+F 2 "" H 7600 5700 60  0000 C CNN
+F 3 "" H 7600 5700 60  0000 C CNN
+	1    7600 5700
+	-1   0    0    1
+$EndComp
+$Comp
+L conservify:PWR_FLAG #FLG0101
+U 1 1 5DA418D8
+P 7200 5850
+F 0 "#FLG0101" H 7200 5925 50  0001 C CNN
+F 1 "PWR_FLAG" H 7200 6000 50  0000 C CNN
+F 2 "" H 7200 5850 50  0001 C CNN
+F 3 "~" H 7200 5850 50  0001 C CNN
+	1    7200 5850
+	-1   0    0    1
+$EndComp
+$Comp
+L conservify:PWR_FLAG #FLG0102
+U 1 1 5DA4194A
+P 7600 5850
+F 0 "#FLG0102" H 7600 5925 50  0001 C CNN
+F 1 "PWR_FLAG" H 7600 6000 50  0000 C CNN
+F 2 "" H 7600 5850 50  0001 C CNN
+F 3 "~" H 7600 5850 50  0001 C CNN
+	1    7600 5850
+	-1   0    0    1
+$EndComp
+Wire Wire Line
+	7600 5700 7600 5850
+Wire Wire Line
+	7200 5850 7200 5700
 $EndSCHEMATC

Commit message: Add BNO055 to sensor board. Larger connector.
Parts:
- removed J1: Conn_01x07, conservify:Molex_CLIK-Mate_502386-0770_1x07_P1.25mm_Horizontal, symbol fk-naturalist-sensors-rescue:Conn_01x07
- added C10, C9: 100nF, conservify:CAP-0603, symbol conservify:CAPACITOR_CERAMIC
- added C11, C8: 22pF, conservify:CAP-0603, symbol conservify:CAPACITOR_CERAMIC
- added J1: CONN_01x09, conservify:Molex_CLIK-Mate_502382-0970_1x09_P1.25mm_Vertical, symbol conservify:CONN_01x09
- added R3, R4, R5: 10K, conservify:RES-0603, symbol conservify:RESISTOR
- added U5: BNO055, conservify:BNO055, symbol conservify:BNO055_JACOB
- added Y1: FC-135, conservify:ABS07, symbol conservify:CRYSTAL
- C6, C7: symbol fk-naturalist-sensors-rescue:CAPACITOR-CERAMIC -> conservify:CAPACITOR_CERAMIC
- renumbered M5 to M1, M8 to M2, M1 to M3, M2 to M4, M6 to M5, M9 to M6, M3 to M7, M4 to M8, M7 to M9
Connections:
- net labels added: SCL2, SDA2
- wire segments 70 -> 109
- no-connect marks 10 -> 14
Other:
- note added: "BNO055"

Commit message: Consistency in part values
Parts:
- C1, C2, C3: Critical (none) -> (none); MFN (none) -> Murata Electronics; MFP (none) -> GRM188R71H104KA93D; Notes (none) -> (none); Package (none) -> (none); Source (none) -> ANY; Subsystem (none) -> (none)
- C4, C6: Critical (none) -> (none); MFN (none) -> Taiyo Yuden; MFP (none) -> UMK107BJ105KA-T; Notes (none) -> (none); Package (none) -> (none); Source (none) -> ANY; Subsystem (none) -> (none)
- C5: Critical (none) -> (none); MFN (none) -> Taiyo Yuden; MFP (none) -> LMK107BBJ106KALT; Notes (none) -> (none); Package (none) -> (none); Source (none) -> ANY; Subsystem (none) -> (none)
- C7, R2: Critical (none) -> (none); MFN (none) -> (none); MFP (none) -> (none); Notes (none) -> (none); Package (none) -> (none); Source (none) -> ANY; Subsystem (none) -> (none)
- J1: Critical (none) -> (none); MFN (none) -> Molex; MFP (none) -> 502382-0970; Notes (none) -> (none); Package (none) -> (none); SPN1 (none) -> WM4786CT-ND; Source (none) -> ANY; Subsystem (none) -> (none); Supplier1 (none) -> digikey
- M1, M10, M2, M3, M4, M5, M6, M7, M8, M9: Critical (none) -> (none); MFN (none) -> (none); MFP (none) -> (none); Notes (none) -> (none); Package (none) -> (none); SPN1 (none) -> (none); Source (none) -> ANY; Subsystem (none) -> (none); Supplier1 (none) -> (none)
- R1: Critical (none) -> (none); MFN (none) -> Yageo; MFP (none) -> RC0603FR-0710KL; Notes (none) -> (none); Package (none) -> (none); Source (none) -> ANY; Subsystem (none) -> (none)
- U1: Critical (none) -> (none); MFN (none) -> NXP / Freescale; MFP (none) -> MPL3115A2; Notes (none) -> (none); Package (none) -> (none); Source (none) -> ANY; Subsystem (none) -> (none)
- U2: Critical (none) -> (none); MFN (none) -> Sensirion; MFP (none) -> SHT31-DIS-B; Notes (none) -> (none); Package (none) -> (none); Source (none) -> ANY; Subsystem (none) -> (none)
- U3: Critical (none) -> (none); MFN (none) -> Knowles; MFP (none) -> SPH0645LM4H-B; Notes (none) -> (none); Package (none) -> (none); Source (none) -> ANY; Subsystem (none) -> (none)
- U4: Critical (none) -> (none); MFN (none) -> AMS; MFP (none) -> TSL25911FN; Notes (none) -> (none); Package (none) -> (none); Source (none) -> ANY; Subsystem (none) -> (none)
