File: hardware/sensor-board/fk-naturalist-sensors.sch (KiCad schematic (older format))
At the start: 33 parts, among them J1 CONN_01x09, M1 FIDUCIAL, M10 FIDUCIAL, M2 FIDUCIAL, M3 MOUNT_HOLE, M4 MOUNT_HOLE, M5 FIDUCIAL, M6 FIDUCIAL, M7 MOUNT_HOLE, M8 MOUNT_HOLE, M9 FIDUCIAL, U1 MPL3115A2, U2 SHT31, U3 SPH0645, U4 TSL2591, U5 BNO055, Y1 FC-135

Commit message: Fix SD landing.
Parts:
- C7: spn1 77-VJ0603A221KXXCBC -> (none)
- R2: spn1 71-RCS060368R0FKEA -> (none)

Commit message: Adding pullups to SDA2/SCL2.
Parts:
- added R6, R7: 4.7K, conservify:RES-0603, symbol conservify:RESISTOR
Connections:
- wire segments 109 -> 113
